File: sensnodeTXv3.sch (EAGLE design)
At the start: 36 parts

Commit message: update sensnodeTX and sensbase
Parts:
- removed 3.3V: TJ3965-3.3, artek:TJ3965-3.3
- removed LDR: (no value), SparkFun:M02PTH
- removed R3: 10k, resistor:R-EU_M0805
- added IC1: MCP1703DB, linear:MCP1703DB
- added P3: (no value), SparkFun:M06SIP_LOCK
- 1-WIRE: device SparkFun:M03PTH -> SparkFun:M03LOCK
- BATTERY, SOLAR: device SparkFun:M02PTH -> SparkFun:M02LOCK
- I2C: device SparkFun:M04PTH -> SparkFun:M04LOCK
- UART: device SparkFun:M06SIP -> SparkFun:M06SIP_LOCK
Connections:
- removed net LDR: ATMEGA8/168/328.PC2(ADC2), LDR.2, R3.1
- new net N$5: ATMEGA8/168/328.PC2(ADC2), P3.5
- new net N$9: ATMEGA8/168/328.PD6(AIN0), P3.2
- net +3V3: now also IC1.VO, P3.4; no longer 3.3V.VOUT, LDR.1
- net DIG3/IRQ: now also P3.6
- net GND: now also IC1.GND, P3.3; no longer 3.3V.GND, R3.2
- net VBUS: now also IC1.VI, P3.1; no longer 3.3V.VIN
Other:
- note added: "N+P"
- note added: "Other Pinouts"
- note removed: "Light measure"
- note removed: "Other Pineouts"
- note removed: "Typu N+P"
